Commit message: add inertia

File: description/base.xacro (robot description, xacro)
@@ -2,4 +2,5 @@
 <robot xmlns:xacro="http://www.ros.org/wiki/xacro">
     <xacro:include filename="common_properties.xacro"/>
+    <xacro:include filename="inertia_properties.xacro"/>
     <!-- BASE LINK -->
     <link name="base_link"></link>
@@ -25,4 +26,13 @@
             <material name="white"/>
         </visual>
+        <collision>
+            <origin xyz="0 0 ${chassis_body_height/2}"/>
+            <geometry>
+                <box size="${chassis_length} ${chassis_width} ${chassis_body_height}"/>
+            </geometry>
+        </collision>
+        <xacro:cuboid_inertia mass="0.6" width="${chassis_width}" height="${chassis_body_height}" depth="${chassis_length}">
+            <origin xyz="0 0 ${chassis_body_height/2}"/>
+        </xacro:cuboid_inertia>
     </link>
     <!-- FRONT LEFT WHEEL -->
@@ -40,4 +50,12 @@
             <material name="black"/>
         </visual>
+        <collision>
+            <geometry>
+                <cylinder radius="${wheel_radius}" length="${wheel_thickness}"/>
+            </geometry>
+        </collision>
+        <xacro:cylinder_inertia mass="0.1" radius="${wheel_radius}" height="${wheel_thickness}">
+            <origin xyz="0 0 0" rpy="0 0 0"/>
+        </xacro:cylinder_inertia>
     </link>
     <!-- FRONT RIGHT WHEEL -->
@@ -55,4 +73,12 @@
             <material name="black"/>
         </visual>
+        <collision>
+            <geometry>
+                <cylinder radius="${wheel_radius}" length="${wheel_thickness}"/>
+            </geometry>
+        </collision>
+        <xacro:cylinder_inertia mass="0.1" radius="${wheel_radius}" height="${wheel_thickness}">
+            <origin xyz="0 0 0" rpy="0 0 0"/>
+        </xacro:cylinder_inertia>
     </link>
     <!-- BACK LEFT WHEEL -->
@@ -70,4 +96,12 @@
             <material name="black"/>
         </visual>
+        <collision>
+            <geometry>
+                <cylinder radius="${wheel_radius}" length="${wheel_thickness}"/>
+            </geometry>
+        </collision>
+        <xacro:cylinder_inertia mass="0.1" radius="${wheel_radius}" height="${wheel_thickness}">
+            <origin xyz="0 0 0" rpy="0 0 0"/>
+        </xacro:cylinder_inertia>
     </link>
     <!-- BACK RIGHT WHEEL -->
@@ -85,4 +119,12 @@
             <material name="black"/>
         </visual>
+        <collision>
+            <geometry>
+                <cylinder radius="${wheel_radius}" length="${wheel_thickness}"/>
+            </geometry>
+        </collision>
+        <xacro:cylinder_inertia mass="0.1" radius="${wheel_radius}" height="${wheel_thickness}">
+            <origin xyz="0 0 0" rpy="0 0 0"/>
+        </xacro:cylinder_inertia>
     </link>
 </robot>

Commit message: Added basic keyboard control

File: description/base.xacro (robot description, xacro)
@@ -3,4 +3,5 @@
     <xacro:include filename="common_properties.xacro"/>
     <xacro:include filename="inertia_properties.xacro"/>
+    <xacro:include filename="gazebo_control.xacro"/>
     <!-- BASE LINK -->
     <link name="base_link"></link>
@@ -36,95 +37,41 @@
         </xacro:cuboid_inertia>
     </link>
-    <!-- FRONT LEFT WHEEL -->
-    <joint name="front_left_wheel_joint" type="continuous">
-        <parent link="base_link"/>
-        <child link="front_left_wheel"/>
-        <origin xyz="${wheel_front_x} ${wheel_y} ${wheel_z}" rpy="-${pi/2} 0 0"/>
-        <axis xyz="0 0 1"/>
-    </joint>
-    <link name="front_left_wheel">
-        <visual>
-            <geometry>
-                <cylinder radius="${wheel_radius}" length="${wheel_thickness}"/>
-            </geometry>
-            <material name="black"/>
-        </visual>
-        <collision>
-            <geometry>
-                <cylinder radius="${wheel_radius}" length="${wheel_thickness}"/>
-            </geometry>
-        </collision>
-        <xacro:cylinder_inertia mass="0.1" radius="${wheel_radius}" height="${wheel_thickness}">
-            <origin xyz="0 0 0" rpy="0 0 0"/>
-        </xacro:cylinder_inertia>
-    </link>
-    <!-- FRONT RIGHT WHEEL -->
-    <joint name="front_right_wheel_joint" type="continuous">
-        <parent link="base_link"/>
-        <child link="front_right_wheel"/>
-        <origin xyz="${wheel_front_x} -${wheel_y} ${wheel_z}" rpy="${pi/2} 0 0"/>
-        <axis xyz="0 0 1"/>
-    </joint>
-    <link name="front_right_wheel">
-        <visual>
-            <geometry>
-                <cylinder radius="${wheel_radius}" length="${wheel_thickness}"/>
-            </geometry>
-            <material name="black"/>
-        </visual>
-        <collision>
-            <geometry>
-                <cylinder radius="${wheel_radius}" length="${wheel_thickness}"/>
-            </geometry>
-        </collision>
-        <xacro:cylinder_inertia mass="0.1" radius="${wheel_radius}" height="${wheel_thickness}">
-            <origin xyz="0 0 0" rpy="0 0 0"/>
-        </xacro:cylinder_inertia>
-    </link>
-    <!-- BACK LEFT WHEEL -->
-    <joint name="back_left_wheel_joint" type="continuous">
-        <parent link="base_link"/>
-        <child link="back_left_wheel"/>
-        <origin xyz="${wheel_back_x} ${wheel_y} ${wheel_z}" rpy="-${pi/2} 0 0"/>
-        <axis xyz="0 0 1"/>
-    </joint>
-    <link name="back_left_wheel">
-        <visual>
-            <geometry>
-                <cylinder radius="${wheel_radius}" length="${wheel_thickness}"/>
-            </geometry>
-            <material name="black"/>
-        </visual>
-        <collision>
-            <geometry>
-                <cylinder radius="${wheel_radius}" length="${wheel_thickness}"/>
-            </geometry>
-        </collision>
-        <xacro:cylinder_inertia mass="0.1" radius="${wheel_radius}" height="${wheel_thickness}">
-            <origin xyz="0 0 0" rpy="0 0 0"/>
-        </xacro:cylinder_inertia>
-    </link>
-    <!-- BACK RIGHT WHEEL -->
-    <joint name="back_right_wheel_joint" type="continuous">
-        <parent link="base_link"/>
-        <child link="back_right_wheel"/>
-        <origin xyz="${wheel_back_x} -${wheel_y} ${wheel_z}" rpy="${pi/2} 0 0"/>
-        <axis xyz="0 0 1"/>
-    </joint>
-    <link name="back_right_wheel">
-        <visual>
-            <geometry>
-                <cylinder radius="${wheel_radius}" length="${wheel_thickness}"/>
-            </geometry>
-            <material name="black"/>
-        </visual>
-        <collision>
-            <geometry>
-                <cylinder radius="${wheel_radius}" length="${wheel_thickness}"/>
-            </geometry>
-        </collision>
-        <xacro:cylinder_inertia mass="0.1" radius="${wheel_radius}" height="${wheel_thickness}">
-            <origin xyz="0 0 0" rpy="0 0 0"/>
-        </xacro:cylinder_inertia>
-    </link>
+    <!-- WHEELS -->
+    <xacro:macro name="wheel" params="prefix x_reflect y_reflect">
+        <link name="${prefix}_wheel">
+            <visual>
+                <geometry>
+                    <cylinder radius="${wheel_radius}" length="${wheel_thickness}"/>
+                </geometry>
+                <material name="black"/>
+            </visual>
+            <collision>
+                <geometry>
+                    <cylinder radius="${wheel_radius}" length="${wheel_thickness}"/>
+                </geometry>
+                <surface>
+                    <friction>
+                        <ode>
+                            <mu>1.0</mu>
+                            <mu2>1.0</mu2>
+                        </ode>
+                    </friction>
+                </surface>
+            </collision>
+            <xacro:cylinder_inertia mass="0.1" radius="${wheel_radius}" height="${wheel_thickness}">
+                <origin xyz="0 0 0" rpy="0 0 0"/>
+            </xacro:cylinder_inertia>
+        </link>
+        <joint name="${prefix}_wheel_joint" type="continuous">
+            <parent link="base_link"/>
+            <child link="${prefix}_wheel"/>
+            <origin xyz="${wheel_offset_x * x_reflect} ${wheel_offset_y * y_reflect} ${wheel_offset_z}" rpy="${-pi/2} 0 0"/>
+            <axis xyz="0 0 1"/>
+            <dynamics damping="${wheel_joint_damping}" friction="${wheel_joint_friction}"/>
+        </joint>
+    </xacro:macro>
+    <xacro:wheel prefix="front_left"  x_reflect="1"  y_reflect="1" />
+    <xacro:wheel prefix="front_right" x_reflect="1"  y_reflect="-1" />
+    <xacro:wheel prefix="back_left"   x_reflect="-1" y_reflect="1" />
+    <xacro:wheel prefix="back_right"  x_reflect="-1" y_reflect="-1" />
 </robot>

File: description/common_properties.xacro (robot description, xacro)
@@ -1,5 +1,5 @@
 <?xml version="1.0"?>
 <robot xmlns:xacro="http://www.ros.org/wiki/xacro">
-    <!-- Geometric properties -->
+    <!-- Geometrics -->
     <xacro:property name="chassis_length" value="0.194"/>
     <xacro:property name="chassis_width"  value="0.168"/>
@@ -9,11 +9,15 @@
     <xacro:property name="wheel_thickness" value="0.0425"/>
     <!-- Offsets -->
-    <xacro:property name="wheel_front_x" value="0.088"/>
-    <xacro:property name="wheel_back_x" value="-0.088"/>
-    <xacro:property name="wheel_y" value="0.105"/>
-    <xacro:property name="wheel_z" value="0.040"/>
+    <xacro:property name="wheel_offset_x" value="0.088"/>
+    <xacro:property name="wheel_offset_y" value="0.105"/>
+    <xacro:property name="wheel_offset_z" value="0.040"/>
+    <!-- Controls -->
+    <xacro:property name="wheel_joint_damping" value="0.1"/>
+    <xacro:property name="wheel_joint_friction" value="0.05"/>
+    <xacro:property name="max_wheel_velocity" value="1.0"/>
+    <xacro:property name="max_wheel_acceleration" value="1.0"/>
     <!-- Materials -->
     <material name="white"> <color rgba="1 1 1 1"/> </material>
     <material name="black"> <color rgba="0 0 0 1"/> </material>
-    <material name="red"> <color rgba="1 0 0 1"/> </material>
+    <material name="red">   <color rgba="1 0 0 1"/> </material>
 </robot>
